File: development/10_KiCAD FC/MoGliFC/MoGliFC.kicad_sch (KiCad schematic)
At the start: 109 parts, among them J1 CAM, J10 RX3, J11 TX3, J12 RX4, J13 TX4, J14 RX5, J15 TX5, J2 OSD, J3 Vid, J4 vA, J5 vRSSI, J6 vAIR, J7 vU, J8 RX1, J9 TX1

Commit message: update
Connections:
- net 5V_BEC renamed 5V_BEC_FC
Other:
- added sheet Power (untitled.kicad_sch)
- note removed: "FC: BAT->5V@2.5A: TPSM33625RDNR"
- note removed: "ToDo: - 10V / 2A - optionally connected to PINIO driven pit switches, and/or jumper pad setups that enable end users to select constant-on or transistor switched behavior, particularly if located to support video transmission systems."
- note removed: "VTX: BAT->10V@2A (DJI:~1A@9V)"
- note removed: "Vx: BAT->5V/6V@4A:"

Commit message: schematic update
Parts:
- removed C1_LDO1, C1_LDO2: 10u, Capacitor_SMD:C_0805_2012Metric, symbol Device:C_Small
- removed C2_LDO1, C2_LDO2: 20u, Capacitor_SMD:C_0805_2012Metric, symbol Device:C_Small
- removed D1, D2: B5819W, Diode_SMD:D_SOD-123, symbol Device:D_Schottky_Small
- removed J_USB1: U263-241N-4BQC11-1, U263241N4BQC111, symbol custom_Library:U263-241N-4BQC11-1
- removed R1, R2: 22, Resistor_SMD:R_0402_1005Metric, symbol Device:R_Small
- removed U_LDO1, U_LDO2: LP5912-3.3DRVR, custom_Library:LP59123.3_SON65P200X200X80-7N, symbol custom_Library:LP5912-3.3DRVR
- removed U_MCU1: STM32H743VITx, Package_QFP:LQFP-100_14x14mm_P0.5mm, symbol MCU_ST_STM32H7:STM32H743VITx
- added R7, R8: 22, Resistor_SMD:R_0402_1005Metric, symbol Device:R_Small
- added U1: STM32H743VIHx, Package_BGA:TFBGA-100_8x8mm_Layout10x10_P0.8mm, symbol MCU_ST_STM32H7:STM32H743VIHx
- added USB_FC1: U262-16XN-4BVC11, custom_Library:USB-3.1-SMD_U262-161N-4BVC11, symbol custom_Library:U262-16XN-4BVC11
Connections:
- net +5V: now also C_can1.1; no longer C_can1.2
- net 3V3_MCU: now also U1.B2 (VBAT), U1.D2 (VDD), U1.F4 (VDDLDO), U1.F5 (VDD), U1.F6 (VDD33_USB), U1.F7 (PDR_ON), U1.H1 (VDDA), U1.K1 (VDD)
- net 5V_USB: now also USB_FC1.A4B9 (VBUS), USB_FC1.B4A9 (VBUS)
- net ADC_CH1_VBAT_ADC3: now also U1.F2 (PC1)
- net ADC_CH2_CURR_ADC3: now also U1.F3 (PC3_C)
- net ADC_CH3_RSSI_ADC3: now also U1.E2 (PC2_C)
- net ADC_CH4_AirS_ADC3: now also U1.F1 (PC0)
- net AT7456_CS_PIN: now also U1.K8 (PB12)
- net BEEPER: now also U1.B3 (PE3)
- net BMI270_CS_PIN: now also U1.G3 (PA4)
- net BOOT0: now also U1.D5 (BOOT0)
- net FDCAN1_RX: now also U1.D8 (PD0)
- net FDCAN1_TX: now also U1.E8 (PD1)
- net GND: now also C_can1.2, U1.C2 (VSS), U1.E4 (VSS), U1.E5 (VSS), U1.E6 (VSS), U1.G1 (VSSA), U1.J1 (VSS), USB_FC1.8 (GND), USB_FC1.A1B12 (GND), USB_FC1.SHELL; no longer C_can1.1, R_can1.1
- net I2C1_SCL: now also U1.B5 (PB6)
- net I2C1_SDA: now also U1.A5 (PB7)
- net LED_0: now also U1.D3 (PE5)
- net LED_1: now also U1.C3 (PE4)
- net NRST: now also U1.E1 (NRST)
- net PINIO_CAM: now also U1.G9 (PD11)
- net PINIO_VTX: now also U1.H9 (PD10)
- net PWM_1: now also U1.G2 (PA0)
- net PWM_2: now also U1.H2 (PA1)
- net PWM_3: now also U1.J2 (PA2)
- net PWM_4: now also U1.K2 (PA3)
- net PWM_5: now also U1.J4 (PB0)
- net PWM_6: now also U1.K4 (PB1)
- net PWM_7: now also U1.F9 (PC8)
- net PWM_8: now also U1.E9 (PC9)
- net SPI1_MISO_PIN : now also U1.J3 (PA6)
- net SPI1_MOSI_PIN: now also U1.K3 (PA7)
- net SPI1_SCK_PIN: now also U1.H3 (PA5)
- net SPI2_MISO_PIN : now also U1.H10 (PB14)
- net SPI2_MOSI_PIN: now also U1.G10 (PB15)
- net SPI2_SCK_PIN: now also U1.J8 (PB13)
- net SPI3_MISO_PIN : now also U1.B8 (PC11)
- net SPI3_MOSI_PIN: now also U1.G5 (PB2)
- net SPI3_NSS_PIN: now also U1.A8 (PA15)
- net SPI3_SCK_PIN: now also U1.B9 (PC10)
- net SWCLK: now also U1.A9 (PA14)
- net SWDIO: now also U1.A10 (PA13)
- net UART1_RX_PIN: now also U1.D10 (PA10)
- net UART1_TX_PIN: now also U1.C9 (PA9)
- net UART2_RX_PIN: now also U1.C6 (PD6)
- net UART2_TX_PIN: now also U1.B6 (PD5)
- net UART3_RX_PIN: now also U1.J9 (PD9)
- net UART3_TX_PIN: now also U1.K9 (PD8)
- net UART4_RX_PIN: now also U1.B4 (PB8)
- net UART4_TX_PIN: now also U1.A4 (PB9)
- net UART5_RX_PIN: now also U1.B7 (PD2)
- net UART5_TX_PIN: now also U1.C8 (PC12)
- net UART6_RX_PIN: now also U1.E10 (PC7)
- net UART6_TX_PIN: now also U1.F10 (PC6)
- net UART7_RX_PIN: now also U1.H5 (PE7)
- net UART7_TX_PIN: now also U1.J5 (PE8)
- net UART8_RX_PIN: now also U1.D4 (PE0)
- net UART8_TX_PIN: now also U1.C4 (PE1)
- net USB+: now also R8.1, USB_FC1.A6 (DP1), USB_FC1.B6 (DP2)
- net USB-: now also R7.1, USB_FC1.A7 (DN1), USB_FC1.B7 (DN2)
- net USB_FS_D+: now also R8.2, U1.B10 (PA12)
- net USB_FS_D-: now also R7.2, U1.C10 (PA11)
- net WS2811_LED_PIN: now also U1.D9 (PA8)
- net vcap1: now also U1.E7 (VCAP)
- net vcap2: now also U1.F8 (VCAP)
- net at R3.1: now also USB_FC1.A5 (CC1)
- net at R4.2: now also USB_FC1.B5 (CC2)
- net led1-: now reaches D_g1.1 (K), R_g1.2
- net MAGset: now reaches C_mag3.2, U_MAG1.8 (SETP)
- net led0-: now reaches D_b1.1 (K), R_b1.2
- net led3V3-: now reaches D_red_3V3.1 (K), R_r1.2
- net at Y_MCU1.1: now also U1.C1 (PH0)
- net at Y_MCU1.3: now also U1.D1 (PH1)
- net I2C2_SCL renamed I2C2_SCL_ext
- net I2C2_SCL_ext: now also U1.J7 (PB10)
- net I2C2_SDA renamed I2C2_SDA_ext
- net I2C2_SDA_ext: now also U1.K7 (PB11)
- new net CANFD_CONTROL_S: R_can1.1, U1.J10 (PD13)
- no-connect marks 49 -> 39
Other:
- note added: "LSC C319148 Shell to ground? Check: TVS dioden C15999?"
- note added: "SPI3: BlackBox 128MByte"
- note added: "USB FC"
- note removed: "- Ref. schematic: CUAV https://github.com/cuav/hardware/tree/master/X7_Autopilot"
- note removed: "3.3V rail 1: 5V->3.3V LDO - MCU --> max.500mA"
- note removed: "3.3V rail 2: 5V->3.3V LDO - onboard max. 140mA(OSD) + ??? - offboard (GPS,...): <100mA --> max xxxmA"
- note removed: "Change: - vertical --> horizontal connector C167321 Check: TVS dioden C15999?"
- note removed: "Goal: - Peak to peak noise: <50mV - PSRR >70dB down as low as 1Hz"
- note removed: "Power Circuitry 5V -> 3.3V"
- note removed: "SPI3: BlackBox 128MByte (xx mA)"
- note removed: "USB"
- moved on the sheet: C_RESET1, C_can1, C_can2, C_can3, R4, R_b1, R_can1, R_can2, R_can3, R_g1, R_r1, U_can1

Commit message: update all
Parts:
- removed J7: vU, Momo footprints Library:PinHeader_1x01_P2.54mm_Vertical, symbol Connector_Generic:Conn_01x01
- C1: # Footprint checked (none) -> -; # Value checked (none) -> -; #LCSC Check (none) -> -; #LCSC Part (none) -> C1532; AVAILABILITY x -> (none); LCSC Part # C1532 -> (none); Price (none) -> -
- CON_pwm1, CON_pwm2, CON_pwm3, CON_pwm4, CON_pwm5, CON_pwm6, CON_pwm7, CON_pwm8, J1, J10, J11, J12, J13, J14, J15, J3, J4, J5, J6, J8, J9: # Footprint checked (none) -> -; # Value checked (none) -> -; #LCSC Check (none) -> -; #LCSC Part (none) -> empty; AVAILABILITY x -> (none); JLCPCB BOM 0 -> (none); LCSC Part # empty -> (none); Price (none) -> -
- C_OSD1, C_OSD2, C_OSD3, C_RESET1, C_STM2, C_STM3, C_STM4, C_STM5, C_STM6, C_STM7, C_STM8, C_can1, C_can2, C_dps1, C_dps2, C_flash1, C_imu1, C_imu2, C_mag1: # Footprint checked (none) -> -; # Value checked (none) -> -; #LCSC Check (none) -> -; #LCSC Part (none) -> C1525; AVAILABILITY x -> (none); LCSC Part # C1525 -> (none); Price (none) -> -
- C_STM1: # Footprint checked (none) -> -; # Value checked (none) -> -; #LCSC Check (none) -> -; #LCSC Part (none) -> C19666; AVAILABILITY x -> (none); LCSC Part # C19666 -> (none); Price (none) -> -
- C_can3: # Footprint checked (none) -> -; # Value checked (none) -> -; #LCSC Check (none) -> -; #LCSC Part (none) -> -; AVAILABILITY x -> (none); LCSC Part # - -> (none); Price (none) -> -
- C_mag2: # Footprint checked (none) -> -; # Value checked (none) -> -; #LCSC Check (none) -> -; #LCSC Part (none) -> C23733; AVAILABILITY x -> (none); LCSC Part # C23733 -> (none); Price (none) -> -
- C_mag3: # Footprint checked (none) -> -; # Value checked (none) -> -; #LCSC Check (none) -> -; #LCSC Part (none) -> C16772; AVAILABILITY x -> (none); LCSC Part # C16772 -> (none); Price (none) -> -
- C_osd4: # Footprint checked (none) -> -; # Value checked (none) -> -; #LCSC Check (none) -> -; #LCSC Part (none) -> C14663; AVAILABILITY x -> (none); JLCPCB xx -> (none); LCSC Part # C14663 -> (none); Price (none) -> -
- C_osd5, C_osd6: # Footprint checked (none) -> -; # Value checked (none) -> -; #LCSC Check (none) -> -; #LCSC Part (none) -> C59461; AVAILABILITY x -> (none); LCSC Part # C59461 -> (none); Price (none) -> -
- C_vcap1, C_vcap2: # Footprint checked (none) -> -; # Value checked (none) -> -; #LCSC Check (none) -> -; #LCSC Part (none) -> C23630; AVAILABILITY x -> (none); LCSC Part # C23630 -> (none); Price (none) -> -
- D_b1: # Footprint checked (none) -> -; # Value checked (none) -> -; #LCSC Check (none) -> -; #LCSC Part (none) -> C72041; AVAILABILITY x -> (none); LCSC Part # C72041 -> (none); Price (none) -> -
- D_g1: # Footprint checked (none) -> -; # Value checked (none) -> -; #LCSC Check (none) -> -; #LCSC Part (none) -> C72043; AVAILABILITY x -> (none); LCSC Part # C72043 -> (none); Price (none) -> -
- D_red_3V3: # Footprint checked (none) -> -; # Value checked (none) -> -; #LCSC Check (none) -> -; #LCSC Part (none) -> C2286; AVAILABILITY x -> (none); LCSC Part # C2286 -> (none); Price (none) -> -
- J_OSD1: renamed from J2; # Footprint checked (none) -> -; # Value checked (none) -> -; #LCSC Check (none) -> -; #LCSC Part (none) -> empty; AVAILABILITY x -> (none); JLCPCB BOM 0 -> (none); LCSC Part # empty -> (none); Price (none) -> -
- R10, R11, R12, R13, R14, R5, R6, R9: # Footprint checked (none) -> -; # Value checked (none) -> -; #LCSC Check (none) -> -; #LCSC Part (none) -> C25087; AVAILABILITY x -> (none); LCSC Part # C25087 -> (none); Price (none) -> -
- R1_i2c1, R1_i2c2, R2_i2c1, R2_i2c2: # Footprint checked (none) -> -; # Value checked (none) -> -; #LCSC Check (none) -> -; #LCSC Part (none) -> C25900; AVAILABILITY x -> (none); LCSC Part # C25900 -> (none); Price (none) -> -
- R3, R4: # Footprint checked (none) -> -; # Value checked (none) -> -; #LCSC Check (none) -> -; #LCSC Part (none) -> C25905; AVAILABILITY x -> (none); LCSC Part # C25905 -> (none); Price (none) -> -
- R7, R8: # Footprint checked (none) -> -; # Value checked (none) -> -; #LCSC Check (none) -> -; #LCSC Part (none) -> C25092; AVAILABILITY x -> (none); LCSC Part # C25092 -> (none); Price (none) -> -
- R_J1, R_can1, R_flash1, R_flash2: # Footprint checked (none) -> -; # Value checked (none) -> -; #LCSC Check (none) -> -; #LCSC Part (none) -> C25744; AVAILABILITY x -> (none); LCSC Part # C25744 -> (none); Price (none) -> -
- R_adc1, R_adc2, R_b1, R_g1, R_r1: # Footprint checked (none) -> -; # Value checked (none) -> -; #LCSC Check (none) -> -; Price (none) -> -
- R_beep1, R_ws2811: # Footprint checked (none) -> -; # Value checked (none) -> -; #LCSC Check (none) -> -; #LCSC Part (none) -> C8218; AVAILABILITY x -> (none); LCSC Part # C8218 -> (none); Price (none) -> -
- R_can2, R_can3: # Footprint checked (none) -> -; # Value checked (none) -> -; #LCSC Check (none) -> -; AVAILABILITY x -> (none); Price (none) -> -
- R_osd1, R_osd2: # Footprint checked (none) -> -; # Value checked (none) -> -; #LCSC Check (none) -> -; #LCSC Part (none) -> C25133; AVAILABILITY x -> (none); LCSC Part # C25133 -> (none); Price (none) -> -
- SW_boot1: # Footprint checked (none) -> -; # Value checked (none) -> -; #LCSC Check (none) -> -; #LCSC Part (none) -> C145874; LCSC Part # C145874 -> (none); Price (none) -> -
- TP1, TP2, TP3, TP4: # Footprint checked (none) -> -; # Value checked (none) -> -; #LCSC Check (none) -> -; #LCSC Part (none) -> -; AVAILABILITY x -> (none); JLCPCB BOM 0 -> (none); LCSC Part # - -> (none); Price (none) -> -
- USB_FC1: # Footprint checked (none) -> -; # Value checked (none) -> -; #LCSC Check (none) -> -; #LCSC Part (none) -> C319148; LCSC Part C319148 -> (none); Price (none) -> -
- U_BARO1: # Footprint checked (none) -> -; # Value checked (none) -> -; #LCSC Check (none) -> -; #LCSC Part (none) -> -; AVAILABILITY Unavailable -> (none); LCSC Part # - -> (none); Price (none) -> -
- U_IMU1, U_flash1: # Footprint checked (none) -> -; # Value checked (none) -> -; #LCSC Check (none) -> -; #LCSC Part (none) -> -; Availability In Stock -> (none); LCSC Part # - -> (none); Price None -> -
- U_MAG1, U_OSD1, U_can1, Y_MCU1, Y_osd1: # Footprint checked (none) -> -; # Value checked (none) -> -; #LCSC Check (none) -> -; #LCSC Part (none) -> -; LCSC Part # - -> (none); Price (none) -> -
- U_STM32: renamed from U1; # Footprint checked (none) -> -; # Value checked (none) -> -; #LCSC Check (none) -> -; Price (none) -> -
Connections:
- net 3V3_MCU: no longer C_STM1.1, C_STM2.1, C_STM3.1, C_STM4.1, C_STM5.1, C_STM6.1, C_STM7.1, C_STM8.1, C_flash1.1, D_red_3V3.2 (A), R_flash1.1, R_flash2.1, SW_boot1.3 (B), SW_boot1.4 (B), U_STM32.B2 (VBAT), U_STM32.D2 (VDD), U_STM32.F4 (VDDLDO), U_STM32.F5 (VDD), U_STM32.F6 (VDD33_USB), U_STM32.H1 (VDDA), U_STM32.K1 (VDD), U_flash1.8 (VCC)
- net SPI3_MOSI_PIN: now also U_STM32.C5 (PB5); no longer U_STM32.G5 (PB2)
- net +5V renamed 5V_BUS
- net 3V3_SENS renamed 3V3_IMU
- net 3V3_IMU: no longer J_OSD1.2 (Pin_2), R1_i2c1.1, R1_i2c2.1, R2_i2c1.1, R2_i2c2.1
- new net 3V3_MCU_OSD: C_STM1.1, C_STM2.1, C_STM3.1, C_STM4.1, C_STM5.1, C_STM6.1, C_STM7.1, C_STM8.1, C_flash1.1, D_red_3V3.2 (A), J_OSD1.2 (Pin_2), R1_i2c1.1, R1_i2c2.1, R2_i2c1.1, R2_i2c2.1, R_flash1.1, R_flash2.1, SW_boot1.3 (B), SW_boot1.4 (B), U_STM32.B2 (VBAT), U_STM32.D2 (VDD), U_STM32.F4 (VDDLDO), U_STM32.F5 (VDD), U_STM32.F6 (VDD33_USB), U_STM32.H1 (VDDA), U_STM32.K1 (VDD), U_flash1.8 (VCC)
- no-connect marks 39 -> 38
Other:
- note added: "Check: - ADC2-4: direct to pin??? - ADC1: voltage scale/divider -airspeedsensor special scaling? 0 - 6V?"
- note removed: "Check: - ADC2-4: direct to pin??? - ADC1: voltage scale/divider"

Commit message: schematic update ELRS
Parts:
- USB_FC1: LCSC Part (none) -> C319148
- U_BARO1: AVAILABILITY (none) -> Unavailable
- U_IMU1, U_flash1: Availability (none) -> In Stock; Price - -> None
Other:
- added sheet expressLRS (expressLRS.kicad_sch)
- moved on the sheet: R_beep1, R_ws2811, TP1, TP2

Commit message: Schematic update
Connections:
- net LED is gone; now on net WS2811_LED_PIN: R_ws2811.1, TP1.1
Other:
- note added: "ToDo: beeper FET"
- moved on the sheet: R_beep1, TP1, TP2
