File: development/10_KiCAD FC/MoGliFC/expressLRS.kicad_sch (KiCad schematic)
At the start: 46 parts, among them SW1 SKTAAAE010, U1 ESP32-PICO-D4, U3 ANT3216LL00R2400A

Commit message: Update expressLRS.kicad_sch
Parts:
- removed C8: 6.2p, Capacitor_SMD:C_0603_1608Metric, symbol Device:C_Small
- added C_pi1: 1p2, Capacitor_SMD:C_0603_1608Metric, symbol Device:C_Small
- added C_pi2: 1p5, Capacitor_SMD:C_0603_1608Metric, symbol Device:C_Small
- added L1: 1n8, symbol Device:L
Connections:
- net GND: now also C_pi1.2, C_pi2.1
- net WIFI_IN: now also C_pi2.2, L1.1
- net at U3.1: now also C_pi1.1, L1.2
Other:
- moved on the sheet: U3

Commit message: Schematic update
Parts:
- removed C_pi2: 1p5, Capacitor_SMD:C_0603_1608Metric, symbol Device:C_Small
- removed L1: 1n8, symbol Device:L
- added R17, R18: 0, Resistor_SMD:R_0402_1005Metric, symbol Device:R
- added R19, R20, R21, R22, R23, R24, R25, R26: 200, Resistor_SMD:R_0402_1005Metric, symbol Device:R_Small
- C_pi1: value 1p2 -> 6.2p; JLCPCB BOM (none) -> xx; LCSC Part # (none) -> C41744
- renumbered C3 to C_ESP1, C5 to C_ESP2, C4 to C_ESP3, C6 to C_ESP4, C7 to C_ESP5, C2 to C_ESP6
Connections:
- net WIFI_IN is gone; now on net wifi_in: U1.2 (LNA_IN)
- net ELRS_RX: now also R22.1
- net ELRS_TX: now also R20.1
- net GND: now also R17.2, R18.2; no longer C_pi1.2
- net boot: now also R19.1
- net wifi_in: now reaches C_pi1.1
- net wifi_in: now also R17.1; no longer U3.1
- net at U1.22 (IO2): now also R21.1
- net at U1.34 (IO5): now also R23.1
- net at U1.35 (IO18): now also R24.1
- net at U1.38 (IO19): now also R25.1
- net at U1.42 (IO21): now also R26.1
- new net PWM_ELRS_1: R19.2
- new net PWM_ELRS_2: R20.2
- new net PWM_ELRS_3: R22.2
- new net PWM_ELRS_4: R26.2
- new net PWM_ELRS_5: R25.2
- new net PWM_ELRS_6: R23.2
- new net PWM_ELRS_7: R21.2
- new net PWM_ELRS_8: R24.2
- new net wifi_out: C_pi1.2, R18.1, U3.1
Other:
- note added: "Integrated ExpressLRS True Diversity RX (PWM: optional)"
- note added: "| Notes: | TBD: additional RF filter"
- note added: "| Notes: | ToDo: ->TXCO"
- note added: "| Notes: | ToDo: update to NEW/available VERSION"
- note added: "| note: | C_pi1: enough for PCB-Antenna | without matching network. | <REV2: substitute with JOHANSON SMD antenna 2450AT18B100E"
- note added: "| note: | PA/LNA: AT2401c or SE2431L"
- note added: "| note: | RXEN can also be set to HIGH all the time"
- note added: "| note: | potential subst:# | - 2450FM07A0029T | - TDK DEA102700LT-6307A2 | - TDK DEA162500LT-1217A1"
- note removed: "C103: enough for PCB-Antenna without matching network. <REV2: substitute with JOHANSON SMD antenna 2450AT18B100E"
- note removed: "ExpressLRS True Diversity RX"
- note removed: "PA/LNA: AT2401c or SE2431L"
- note removed: "RXEN can also be set to HIGH all the time"
- note removed: "potential subst:# - 2450FM07A0029T - TDK DEA102700LT-6307A2 - TDK DEA162500LT-1217A1"
- moved on the sheet: C_ESP2, C_ESP3, C_ESP4, C_ESP5, C_ESP6, R15, SW1, U3
